File: whackamole/whackamole/whackamole.kicad_sch (KiCad schematic)
At the start: 22 parts

Commit message: with sound
Parts:
- removed R13: 100, symbol Device:R
Connections:
- net at N_pwr_swtch.3 (D), R5.2, pwr_switch1.1 (Pin_1): now also P_pwr_swtch.2 (G)
- no-connect marks 13 -> 11
Changed lines of the file:
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@@
   (no_connect (at 41.91 68.58))
   (no_connect (at 67.31 73.66))
-  (no_connect (at 41.91 101.6))
   (no_connect (at 67.31 71.12))
   (no_connect (at 67.31 81.28))
   (no_connect (at 67.31 101.6))
   (no_connect (at 120.65 99.06))
-  (no_connect (at 41.91 99.06))
   (no_connect (at 67.31 104.14))
   (no_connect (at 57.15 60.96))
@@
     (stroke (width 0) (type default))
   )
-  (wire (pts (xy 187.96 142.24) (xy 187.96 134.62))
-    (stroke (width 0) (type default))
-  )
   (wire (pts (xy 125.73 121.92) (xy 161.29 121.92))
     (stroke (width 0) (type default))
@@
     (stroke (width 0) (type default))
   )
+  (wire (pts (xy 189.23 119.38) (xy 189.23 121.92))
+    (stroke (width 0) (type default))
+  )
   (wire (pts (xy 85.09 88.9) (xy 87.63 88.9))
     (stroke (width 0) (type default))
   )
-  (wire (pts (xy 189.23 142.24) (xy 189.23 124.46))
+  (wire (pts (xy 189.23 130.81) (xy 189.23 124.46))
     (stroke (width 0) (type default))
   )
@@
     (stroke (width 0) (type default))
   )
-  (wire (pts (xy 153.67 31.75) (xy 172.72 31.75))
+  (wire (pts (xy 153.67 31.75) (xy 184.15 31.75))
     (stroke (width 0) (type default))
   )
@@
     (stroke (width 0) (type default))
   )
-  (wire (pts (xy 26.67 134.62) (xy 26.67 83.82))
+  (wire (pts (xy 26.67 130.81) (xy 26.67 83.82))
     (stroke (width 0) (type default))
   )
@@
     (stroke (width 0) (type default))
   )
-  (wire (pts (xy 187.96 142.24) (xy 189.23 142.24))
+  (wire (pts (xy 26.67 130.81) (xy 189.23 130.81))
     (stroke (width 0) (type default))
   )
@@
     (stroke (width 0) (type default))
   )
-  (wire (pts (xy 189.23 119.38) (xy 189.23 121.92))
-    (stroke (width 0) (type default))
-  )
   (wire (pts (xy 100.33 81.28) (xy 95.25 81.28))
     (stroke (width 0) (type default))
@@
     (stroke (width 0) (type default))
   )
-  (wire (pts (xy 180.34 31.75) (xy 184.15 31.75))
-    (stroke (width 0) (type default))
-  )
   (wire (pts (xy 38.1 116.84) (xy 38.1 93.98))
     (stroke (width 0) (type default))
@@
   )
   (wire (pts (xy 153.67 27.94) (xy 153.67 29.21))
-    (stroke (width 0) (type default))
-  )
-  (wire (pts (xy 26.67 134.62) (xy 187.96 134.62))
     (stroke (width 0) (type default))
   )
@@
         )
       )
-    )
-  )
-  (symbol (lib_id "Device:R") (at 176.53 31.75 90) (unit 1)
-    (in_bom yes) (on_board yes) (dnp no) (fields_autoplaced)
-    (property "Reference" "R13" (at 176.53 25.4 90)
-      (effects (font (size 1.27 1.27)))
-    )
-    (property "Value" "100" (at 176.53 27.94 90)
-      (effects (font (size 1.27 1.27)))
-    )
-    (property "Footprint" "" (at 176.53 33.528 90)
-      (effects (font (size 1.27 1.27)) hide)
-    )
-    (property "Datasheet" "~" (at 176.53 31.75 0)
-      (effects (font (size 1.27 1.27)) hide)
-    )
-    (pin "2")
-    (pin "1")
-    (instances
-      (project "whackamole"
-        (path "/c1d152d8-520f-4b1f-be58-40784473a3d2"
-          (reference "R13") (unit 1)
-        )
-      )
