File: whackamole/whackamole/_autosave-whackamole.kicad_sch (KiCad schematic)
At the start: 20 parts

Commit message: wip save
Parts:
- added D1: 1N4148, Diode_THT:D_DO-35_SOD27_P7.62mm_Horizontal, symbol Diode:1N4148
Connections:
- net +6V: now also D1.2 (A); no longer P_pwr_swtch1.1 (D), R13.1
- net at Arduino_nano1.24 (SCL/A5): now also btn_out1.10 (Pin_10), btn_out1.6 (Pin_6), btn_out1.7 (Pin_7), btn_out1.8 (Pin_8), btn_out1.9 (Pin_9)
- new net: D1.1 (K), P_pwr_swtch1.1 (D), R13.1
- now unconnected: Arduino_nano1.9 (D6)
Changed lines of the file:
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@@
   (junction (at 279.4 44.45) (diameter 0) (color 0 0 0 0)
   )
-  (no_connect (at 120.65 99.06))
   (no_connect (at 55.88 119.38))
   (no_connect (at 30.48 129.54))
@@
   (no_connect (at 30.48 127))
   (no_connect (at 120.65 71.12))
+  (no_connect (at 95.25 83.82))
   (no_connect (at 120.65 81.28))
   (no_connect (at 120.65 101.6))
@@
     (stroke (width 0) (type default))
   )
+  (wire (pts (xy 222.25 130.81) (xy 124.46 130.81))
+    (stroke (width 0) (type default))
+  )
   (wire (pts (xy 222.25 104.14) (xy 222.25 106.68))
     (stroke (width 0) (type default))
@@
     (stroke (width 0) (type default))
   )
-  (wire (pts (xy 82.55 83.82) (xy 95.25 83.82))
-    (stroke (width 0) (type default))
-  )
   (wire (pts (xy 148.59 120.65) (xy 87.63 120.65))
     (stroke (width 0) (type default))
@@
     (stroke (width 0) (type default))
   )
-  (wire (pts (xy 82.55 132.08) (xy 82.55 83.82))
-    (stroke (width 0) (type default))
-  )
   (wire (pts (xy 279.4 30.48) (xy 279.4 44.45))
     (stroke (width 0) (type default))
   )
-  (wire (pts (xy 82.55 132.08) (xy 222.25 132.08))
-    (stroke (width 0) (type default))
-  )
   (wire (pts (xy 85.09 88.9) (xy 95.25 88.9))
     (stroke (width 0) (type default))
@@
     (stroke (width 0) (type default))
   )
+  (wire (pts (xy 124.46 99.06) (xy 120.65 99.06))
+    (stroke (width 0) (type default))
+  )
   (wire (pts (xy 172.72 44.45) (xy 200.66 44.45))
     (stroke (width 0) (type default))
@@
     (stroke (width 0) (type default))
   )
+  (wire (pts (xy 269.24 20.32) (xy 279.4 20.32))
+    (stroke (width 0) (type default))
+  )
   (wire (pts (xy 120.65 86.36) (xy 125.73 86.36))
     (stroke (width 0) (type default))
@@
     (stroke (width 0) (type default))
   )
-  (wire (pts (xy 245.11 20.32) (xy 279.4 20.32))
+  (wire (pts (xy 245.11 20.32) (xy 261.62 20.32))
     (stroke (width 0) (type default))
   )
@@
     (stroke (width 0) (type default))
   )
+  (wire (pts (xy 124.46 130.81) (xy 124.46 99.06))
+    (stroke (width 0) (type default))
+  )
   (wire (pts (xy 153.67 83.82) (xy 147.32 83.82))
     (stroke (width 0) (type default))
@@
     (stroke (width 0) (type default))
   )
+  (wire (pts (xy 222.25 130.81) (xy 222.25 114.3))
+    (stroke (width 0) (type default))
+  )
   (wire (pts (xy 245.11 48.26) (xy 245.11 36.83))
     (stroke (width 0) (type default))
@@
     (stroke (width 0) (type default))
   )
-  (wire (pts (xy 222.25 114.3) (xy 222.25 132.08))
-    (stroke (width 0) (type default))
-  )
   (wire (pts (xy 96.52 73.66) (xy 95.25 73.66))
     (stroke (width 0) (type default))
@@
     (stroke (width 0) (type default))
   )
+  (symbol (lib_id "Diode:1N4148") (at 265.43 20.32 0) (unit 1)
+    (in_bom yes) (on_board yes) (dnp no) (fields_autoplaced)
+    (property "Reference" "D1" (at 265.43 13.97 0)
+      (effects (font (size 1.27 1.27)))
+    )
+    (property "Value" "1N4148" (at 265.43 16.51 0)
+      (effects (font (size 1.27 1.27)))
+    )
+    (property "Footprint" "Diode_THT:D_DO-35_SOD27_P7.62mm_Horizontal" (at 265.43 20.32 0)
+      (effects (font (size 1.27 1.27)) hide)
+    )
+    (property "Datasheet" "https://assets.nexperia.com/documents/data-sheet/1N4148_1N4448.pdf" (at 265.43 20.32 0)
+      (effects (font (size 1.27 1.27)) hide)
+    )
+    (property "Sim.Device" "D" (at 265.43 20.32 0)
+      (effects (font (size 1.27 1.27)) hide)
+    )
+    (property "Sim.Pins" "1=K 2=A" (at 265.43 20.32 0)
+      (effects (font (size 1.27 1.27)) hide)
+    )
+    (pin "2")
+    (pin "1")
+    (instances
+      (project "whackamole"
+        (path "/c1d152d8-520f-4b1f-be58-40784473a3d2"
+          (reference "D1") (unit 1)
+        )
+      )
+    )
+  )
   (symbol (lib_id "MCU_Module:Arduino_Nano_Every") (at 107.95 86.36 0) (unit 1)
