File: bam/bam.kicad_sch (KiCad schematic)
At the start: 18 parts, among them J1 battery, Q1 VP3203N3-G, Q2 PN2222A, SW1 pwr, SW2 next, SW3 play/pause, U1 NE555P

Commit message: true latch
Parts:
- added C3: C_Polarized, symbol Device:C_Polarized
- added Q3: PN2222A, Package_TO_SOT_THT:TO-92_Inline, symbol Transistor_BJT:PN2222A
- added R6: 100k, symbol Device:R
- added R7: 10k, symbol Device:R
- added R8: 100, symbol Device:R
- SW1: value pwr -> on/off
Connections:
- net +5V: now also R6.1
- net GND: now also C3.2, Q3.1 (E); no longer SW1.1
- net at Q2.3 (C), R1.2, R2.1: no longer SW1.2, U1.2 (TR)
- net at R3.1: now also SW1.1, R7.1, R8.1; no longer Q2.2 (B)
- net at R3.2: now also Q2.2 (B); no longer U1.3 (Q)
- new net: Q3.2 (B), R7.2
- new net: C3.1, Q3.3 (C), R6.2, SW1.2
- new net latch: R8.2, U1.3 (Q)
Other:
- moved on the sheet: Q1, Q2, R2

Commit message: wip
Parts:
- R8: value 100 -> 1k
Connections:
- net at Q2.3 (C), R1.2, R2.1: now also U1.2 (TR)
Other:
- moved on the sheet: U3
Changed lines of the file:
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@@
   (junction (at 209.55 55.88) (diameter 0) (color 0 0 0 0)
   )
+  (junction (at 115.57 96.52) (diameter 0) (color 0 0 0 0)
+  )
   (junction (at 163.83 63.5) (diameter 0) (color 0 0 0 0)
   )
   (junction (at 99.06 80.01) (diameter 0) (color 0 0 0 0)
   )
-  (junction (at 163.83 90.17) (diameter 0) (color 0 0 0 0)
-  )
   (junction (at 58.42 96.52) (diameter 0) (color 0 0 0 0)
   )
@@
   )
   (junction (at 99.06 40.64) (diameter 0) (color 0 0 0 0)
+  )
+  (junction (at 163.83 96.52) (diameter 0) (color 0 0 0 0)
   )
   (junction (at 87.63 40.64) (diameter 0) (color 0 0 0 0)
@@
     (stroke (width 0) (type default))
   )
-  (wire (pts (xy 163.83 90.17) (xy 163.83 91.44))
-    (stroke (width 0) (type default))
-  )
   (wire (pts (xy 213.36 78.74) (xy 243.84 78.74))
     (stroke (width 0) (type default))
@@
     (stroke (width 0) (type default))
   )
-  (wire (pts (xy 45.72 40.64) (xy 52.07 40.64))
+  (wire (pts (xy 45.72 40.64) (xy 49.53 40.64))
     (stroke (width 0) (type default))
   )
@@
     (stroke (width 0) (type default))
   )
+  (wire (pts (xy 115.57 96.52) (xy 163.83 96.52))
+    (stroke (width 0) (type default))
+  )
   (wire (pts (xy 99.06 80.01) (xy 99.06 85.09))
     (stroke (width 0) (type default))
@@
     (stroke (width 0) (type default))
   )
-  (wire (pts (xy 195.58 88.9) (xy 195.58 90.17))
-    (stroke (width 0) (type default))
-  )
-  (wire (pts (xy 45.72 43.18) (xy 52.07 43.18))
+  (wire (pts (xy 195.58 88.9) (xy 195.58 96.52))
+    (stroke (width 0) (type default))
+  )
+  (wire (pts (xy 45.72 43.18) (xy 49.53 43.18))
     (stroke (width 0) (type default))
   )
@@
     (stroke (width 0) (type default))
   )
-  (wire (pts (xy 195.58 90.17) (xy 163.83 90.17))
+  (wire (pts (xy 195.58 96.52) (xy 163.83 96.52))
     (stroke (width 0) (type default))
   )
@@
     (stroke (width 0) (type default))
   )
-  (wire (pts (xy 163.83 86.36) (xy 163.83 90.17))
-    (stroke (width 0) (type default))
-  )
-  (wire (pts (xy 101.6 58.42) (xy 87.63 58.42))
-    (stroke (width 0) (type default))
-  )
-  (wire (pts (xy 72.39 40.64) (xy 87.63 40.64))
+  (wire (pts (xy 163.83 86.36) (xy 163.83 96.52))
+    (stroke (width 0) (type default))
+  )
+  (wire (pts (xy 87.63 58.42) (xy 101.6 58.42))
+    (stroke (width 0) (type default))
+  )
+  (wire (pts (xy 151.13 69.85) (xy 151.13 71.12))
+    (stroke (width 0) (type default))
+  )
+  (wire (pts (xy 69.85 40.64) (xy 87.63 40.64))
     (stroke (width 0) (type default))
   )
@@
     (stroke (width 0) (type default))
   )
+  (wire (pts (xy 87.63 69.85) (xy 87.63 58.42))
+    (stroke (width 0) (type default))
+  )
   (wire (pts (xy 179.07 30.48) (xy 190.5 30.48))
     (stroke (width 0) (type default))
@@
     (stroke (width 0) (type default))
   )
-  (wire (pts (xy 72.39 52.07) (xy 45.72 52.07))
+  (wire (pts (xy 69.85 52.07) (xy 45.72 52.07))
     (stroke (width 0) (type default))
   )
@@
     (stroke (width 0) (type default))
   )
+  (wire (pts (xy 151.13 69.85) (xy 87.63 69.85))
+    (stroke (width 0) (type default))
+  )
   (wire (pts (xy 132.08 17.78) (xy 132.08 63.5))
     (stroke (width 0) (type default))
@@
     (stroke (width 0) (type default))
   )
-  (wire (pts (xy 72.39 43.18) (xy 72.39 52.07))
+  (wire (pts (xy 69.85 43.18) (xy 69.85 52.07))
     (stroke (width 0) (type default))
   )
@@
     )
   )
-  (symbol (lib_id "bam:5v-step-up") (at 57.15 48.26 0) (unit 1)
-    (in_bom yes) (on_board yes) (dnp no) (fields_autoplaced)
-    (property "Reference" "U3" (at 62.23 33.02 0)
-      (effects (font (size 1.27 1.27)))
-    )
-    (property "Value" "~" (at 57.15 48.26 0)
-      (effects (font (size 1.27 1.27)))
-    )
-    (property "Footprint" "" (at 57.15 48.26 0)
-      (effects (font (size 1.27 1.27)) hide)
-    )
-    (property "Datasheet" "" (at 57.15 48.26 0)
+  (symbol (lib_id "bam:5v-step-up") (at 54.61 48.26 0) (unit 1)
+    (in_bom yes) (on_board yes) (dnp no) (fields_autoplaced)
+    (property "Reference" "U3" (at 59.69 33.02 0)
+      (effects (font (size 1.27 1.27)))
+    )
+    (property "Value" "~" (at 54.61 48.26 0)
+      (effects (font (size 1.27 1.27)))
+    )
+    (property "Footprint" "" (at 54.61 48.26 0)
+      (effects (font (size 1.27 1.27)) hide)
+    )
+    (property "Datasheet" "" (at 54.61 48.26 0)
       (effects (font (size 1.27 1.27)) hide)
     )
@@
       (effects (font (size 1.27 1.27)) (justify right))
     )
-    (property "Value" "100" (at 80.01 72.39 0)
+    (property "Value" "1k" (at 80.01 72.39 0)
       (effects (font (size 1.27 1.27)) (justify right))
     )
@@
         )
       )
-    )
-  )
-  (symbol (lib_id "power:GND") (at 163.83 91.44 0) (unit 1)
-    (in_bom yes) (on_board yes) (dnp no) (fields_autoplaced)
-    (property "Reference" "#PWR04" (at 163.83 97.79 0)
-      (effects (font (size 1.27 1.27)) hide)
-    )
-    (property "Value" "GND" (at 163.83 96.52 0)
-      (effects (font (size 1.27 1.27)))
-    )
-    (property "Footprint" "" (at 163.83 91.44 0)
-      (effects (font (size 1.27 1.27)) hide)
-    )
-    (property "Datasheet" "" (at 163.83 91.44 0)
-      (effects (font (size 1.27 1.27)) hide)
-    )
-    (pin "1")
-    (instances
-      (project "bam"
-        (path "/81bf8c4d-35fa-42c7-93c2-098e5ef35825"
-          (reference "#PWR04") (unit 1)
-        )
-      )

Commit message: progress
Parts:
- added C4: 3.3uF, symbol Device:C_Polarized
- added R10, R9: 100k, symbol Device:R
- C1: value C_Polarized -> 100uF
- R1: value 100k -> 50k
- R4: value R -> 100k
Connections:
- net GND: now also C4.2
- net at C2.1, Q1.1 (S), R4.1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: now also R10.1
- net at C1.1, D1.2 (A), R4.2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: now also R9.2
- net at Q2.3 (C), R1.2, R2.1: no longer U1.2 (TR)
- new net: C4.1, R10.2, R9.1, U1.2 (TR)
Changed lines of the file:
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@@
   (junction (at 87.63 58.42) (diameter 0) (color 0 0 0 0)
   )
+  (junction (at 139.7 85.09) (diameter 0) (color 0 0 0 0)
+  )
   (junction (at 163.83 46.99) (diameter 0) (color 0 0 0 0)
   )
@@
   (junction (at 66.04 96.52) (diameter 0) (color 0 0 0 0)
   )
+  (junction (at 179.07 81.28) (diameter 0) (color 0 0 0 0)
+  )
   (junction (at 45.72 52.07) (diameter 0) (color 0 0 0 0)
   )
   (junction (at 45.72 40.64) (diameter 0) (color 0 0 0 0)
   )
+  (junction (at 139.7 71.12) (diameter 0) (color 0 0 0 0)
+  )
   (junction (at 209.55 52.07) (diameter 0) (color 0 0 0 0)
   )
@@
   )
   (junction (at 163.83 55.88) (diameter 0) (color 0 0 0 0)
+  )
+  (junction (at 139.7 63.5) (diameter 0) (color 0 0 0 0)
+  )
+  (junction (at 139.7 96.52) (diameter 0) (color 0 0 0 0)
   )
   (junction (at 132.08 63.5) (diameter 0) (color 0 0 0 0)
@@
     (stroke (width 0) (type default))
   )
+  (wire (pts (xy 179.07 81.28) (xy 179.07 91.44))
+    (stroke (width 0) (type default))
+  )
   (wire (pts (xy 99.06 80.01) (xy 115.57 80.01))
     (stroke (width 0) (type default))
   )
+  (wire (pts (xy 151.13 71.12) (xy 139.7 71.12))
+    (stroke (width 0) (type default))
+  )
   (wire (pts (xy 66.04 96.52) (xy 99.06 96.52))
     (stroke (width 0) (type default))
@@
     (stroke (width 0) (type default))
   )
+  (wire (pts (xy 139.7 63.5) (xy 163.83 63.5))
+    (stroke (width 0) (type default))
+  )
   (wire (pts (xy 208.28 52.07) (xy 209.55 52.07))
     (stroke (width 0) (type default))
@@
     (stroke (width 0) (type default))
   )
-  (wire (pts (xy 132.08 63.5) (xy 163.83 63.5))
+  (wire (pts (xy 132.08 63.5) (xy 139.7 63.5))
     (stroke (width 0) (type default))
   )
@@
     (stroke (width 0) (type default))
   )
-  (wire (pts (xy 115.57 96.52) (xy 163.83 96.52))
+  (wire (pts (xy 115.57 96.52) (xy 139.7 96.52))
     (stroke (width 0) (type default))
   )
@@
     (stroke (width 0) (type default))
   )
+  (wire (pts (xy 139.7 85.09) (xy 139.7 86.36))
+    (stroke (width 0) (type default))
+  )
   (wire (pts (xy 190.5 36.83) (xy 196.85 36.83))
     (stroke (width 0) (type default))
@@
     (stroke (width 0) (type default))
   )
+  (wire (pts (xy 171.45 91.44) (xy 149.86 91.44))
+    (stroke (width 0) (type default))
+  )
   (wire (pts (xy 45.72 43.18) (xy 49.53 43.18))
     (stroke (width 0) (type default))
@@
     (stroke (width 0) (type default))
   )
+  (wire (pts (xy 139.7 71.12) (xy 139.7 85.09))
+    (stroke (width 0) (type default))
+  )
   (wire (pts (xy 77.47 74.93) (xy 77.47 80.01))
     (stroke (width 0) (type default))
@@
     (stroke (width 0) (type default))
   )
+  (wire (pts (xy 139.7 93.98) (xy 139.7 96.52))
+    (stroke (width 0) (type default))
+  )
   (wire (pts (xy 163.83 63.5) (xy 163.83 66.04))
     (stroke (width 0) (type default))
@@
     (stroke (width 0) (type default))
   )
-  (wire (pts (xy 151.13 69.85) (xy 151.13 71.12))
-    (stroke (width 0) (type default))
-  )
   (wire (pts (xy 69.85 40.64) (xy 87.63 40.64))
     (stroke (width 0) (type default))
@@
     (stroke (width 0) (type default))
   )
+  (wire (pts (xy 149.86 91.44) (xy 149.86 85.09))
+    (stroke (width 0) (type default))
+  )
   (wire (pts (xy 151.13 81.28) (xy 132.08 81.28))
     (stroke (width 0) (type default))
@@
     (stroke (width 0) (type default))
   )
-  (wire (pts (xy 87.63 69.85) (xy 87.63 58.42))
-    (stroke (width 0) (type default))
-  )
   (wire (pts (xy 179.07 30.48) (xy 190.5 30.48))
     (stroke (width 0) (type default))
@@
     (stroke (width 0) (type default))
   )
+  (wire (pts (xy 139.7 96.52) (xy 163.83 96.52))
+    (stroke (width 0) (type default))
+  )
   (wire (pts (xy 99.06 96.52) (xy 99.06 95.25))
     (stroke (width 0) (type default))
   )
-  (wire (pts (xy 151.13 69.85) (xy 87.63 69.85))
-    (stroke (width 0) (type default))
-  )
   (wire (pts (xy 132.08 17.78) (xy 132.08 63.5))
     (stroke (width 0) (type default))
@@
   )
   (wire (pts (xy 118.11 63.5) (xy 132.08 63.5))
+    (stroke (width 0) (type default))
+  )
+  (wire (pts (xy 149.86 85.09) (xy 139.7 85.09))
     (stroke (width 0) (type default))
   )
@@
     )
   )
+  (symbol (lib_id "Device:R") (at 139.7 67.31 0) (unit 1)
+    (in_bom yes) (on_board yes) (dnp no) (fields_autoplaced)
+    (property "Reference" "R10" (at 142.24 66.04 0)
+      (effects (font (size 1.27 1.27)) (justify left))
+    )
+    (property "Value" "100k" (at 142.24 68.58 0)
+      (effects (font (size 1.27 1.27)) (justify left))
+    )
+    (property "Footprint" "" (at 137.922 67.31 90)
+      (effects (font (size 1.27 1.27)) hide)
+    )
+    (property "Datasheet" "~" (at 139.7 67.31 0)
+      (effects (font (size 1.27 1.27)) hide)
+    )
+    (pin "2")
+    (pin "1")
+    (instances
+      (project "bam"
+        (path "/81bf8c4d-35fa-42c7-93c2-098e5ef35825"
+          (reference "R10") (unit 1)
+        )
+      )
+    )
+  )
   (symbol (lib_id "power:GND") (at 209.55 57.15 0) (unit 1)
     (in_bom yes) (on_board yes) (dnp no) (fields_autoplaced)
@@
         (path "/81bf8c4d-35fa-42c7-93c2-098e5ef35825"
           (reference "#PWR05") (unit 1)
+        )
+      )
+    )
+  )
+  (symbol (lib_id "Device:C_Polarized") (at 139.7 90.17 0) (unit 1)
+    (in_bom yes) (on_board yes) (dnp no) (fields_autoplaced)
+    (property "Reference" "C4" (at 143.51 88.011 0)
+      (effects (font (size 1.27 1.27)) (justify left))
+    )
+    (property "Value" "3.3uF" (at 143.51 90.551 0)
+      (effects (font (size 1.27 1.27)) (justify left))
+    )
+    (property "Footprint" "" (at 140.6652 93.98 0)
+      (effects (font (size 1.27 1.27)) hide)
+    )
+    (property "Datasheet" "~" (at 139.7 90.17 0)
+      (effects (font (size 1.27 1.27)) hide)
+    )
+    (pin "1")
+    (pin "2")
+    (instances
+      (project "bam"
+        (path "/81bf8c4d-35fa-42c7-93c2-098e5ef35825"
+          (reference "C4") (unit 1)
         )
       )
@@
       (effects (font (size 1.27 1.27)) (justify left))
     )
-    (property "Value" "C_Polarized" (at 199.39 85.471 0)
+    (property "Value" "100uF" (at 199.39 85.471 0)
       (effects (font (size 1.27 1.27)) (justify left))
     )
@@
       (effects (font (size 1.27 1.27)) (justify left))
     )
-    (property "Value" "100k" (at 90.17 48.26 0)
+    (property "Value" "50k" (at 90.17 48.26 0)
       (effects (font (size 1.27 1.27)) (justify left))
     )
@@
       (effects (font (size 1.27 1.27)))
     )
-    (property "Value" "R" (at 184.15 59.69 90)
+    (property "Value" "100k" (at 184.15 59.69 90)
       (effects (font (size 1.27 1.27)))
     )
@@
         )
       )
+    )
+  )
+  (symbol (lib_id "Device:R") (at 175.26 91.44 90) (unit 1)
+    (in_bom yes) (on_board yes) (dnp no) (fields_autoplaced)
+    (property "Reference" "R9" (at 175.26 85.09 90)
+      (effects (font (size 1.27 1.27)))
+    )
+    (property "Value" "100k" (at 175.26 87.63 90)
+      (effects (font (size 1.27 1.27)))
+    )
+    (property "Footprint" "" (at 175.26 93.218 90)
+      (effects (font (size 1.27 1.27)) hide)
+    )
+    (property "Datasheet" "~" (at 175.26 91.44 0)
+      (effects (font (size 1.27 1.27)) hide)
+    )
+    (pin "2")
+    (pin "1")
+    (instances
+      (project "bam"
+        (path "/81bf8c4d-35fa-42c7-93c2-098e5ef35825"
+          (reference "R9") (unit 1)
+        )
+      )

Commit message: minor updates
Parts:
- removed R5: 33k, symbol Device:R
- SW3: value play/pause -> previous
Connections:
- net at U2.9 (IO1): now also SW3.2
- net latch renamed keep_alive
Other:
- moved on the sheet: SW2
Changed lines of the file:
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@@
   (junction (at 139.7 85.09) (diameter 0) (color 0 0 0 0)
   )
+  (junction (at 99.06 40.64) (diameter 0) (color 0 0 0 0)
+  )
+  (junction (at 163.83 96.52) (diameter 0) (color 0 0 0 0)
+  )
+  (junction (at 87.63 40.64) (diameter 0) (color 0 0 0 0)
+  )
+  (junction (at 45.72 43.18) (diameter 0) (color 0 0 0 0)
+  )
+  (junction (at 66.04 96.52) (diameter 0) (color 0 0 0 0)
+  )
   (junction (at 163.83 46.99) (diameter 0) (color 0 0 0 0)
   )
-  (junction (at 99.06 40.64) (diameter 0) (color 0 0 0 0)
-  )
-  (junction (at 163.83 96.52) (diameter 0) (color 0 0 0 0)
-  )
-  (junction (at 87.63 40.64) (diameter 0) (color 0 0 0 0)
-  )
-  (junction (at 45.72 43.18) (diameter 0) (color 0 0 0 0)
-  )
-  (junction (at 66.04 96.52) (diameter 0) (color 0 0 0 0)
-  )
   (junction (at 179.07 81.28) (diameter 0) (color 0 0 0 0)
   )
@@
   (junction (at 195.58 78.74) (diameter 0) (color 0 0 0 0)
   )
-  (no_connect (at 196.85 34.29))
   (no_connect (at 196.85 46.99))
   (no_connect (at 151.13 76.2))
@@
   (no_connect (at 196.85 29.21))
   (no_connect (at 222.25 36.83))
+  (no_connect (at 196.85 39.37))
   (wire (pts (xy 58.42 96.52) (xy 66.04 96.52))
     (stroke (width 0) (type default))
@@
     (stroke (width 0) (type default))
   )
-  (wire (pts (xy 163.83 30.48) (xy 168.91 30.48))
+  (wire (pts (xy 163.83 46.99) (xy 168.91 46.99))
     (stroke (width 0) (type default))
   )
@@
     (stroke (width 0) (type default))
   )
-  (wire (pts (xy 163.83 46.99) (xy 168.91 46.99))
-    (stroke (width 0) (type default))
-  )
   (wire (pts (xy 222.25 40.64) (xy 223.52 40.64))
     (stroke (width 0) (type default))
@@
     (stroke (width 0) (type default))
   )
-  (wire (pts (xy 190.5 30.48) (xy 190.5 36.83))
+  (wire (pts (xy 190.5 46.99) (xy 190.5 36.83))
     (stroke (width 0) (type default))
   )
@@
     (stroke (width 0) (type default))
   )
+  (wire (pts (xy 168.91 34.29) (xy 163.83 34.29))
+    (stroke (width 0) (type default))
+  )
   (wire (pts (xy 190.5 36.83) (xy 196.85 36.83))
     (stroke (width 0) (type default))
@@
     (stroke (width 0) (type default))
   )
-  (wire (pts (xy 190.5 39.37) (xy 196.85 39.37))
-    (stroke (width 0) (type default))
-  )
   (wire (pts (xy 77.47 80.01) (xy 85.09 80.01))
     (stroke (width 0) (type default))
@@
     (stroke (width 0) (type default))
   )
+  (wire (pts (xy 163.83 34.29) (xy 163.83 46.99))
+    (stroke (width 0) (type default))
+  )
   (wire (pts (xy 179.07 78.74) (xy 195.58 78.74))
     (stroke (width 0) (type default))
@@
     (stroke (width 0) (type default))
   )
-  (wire (pts (xy 186.69 46.99) (xy 190.5 46.99))
-    (stroke (width 0) (type default))
-  )
   (wire (pts (xy 139.7 93.98) (xy 139.7 96.52))
     (stroke (width 0) (type default))
@@
     (stroke (width 0) (type default))
   )
-  (wire (pts (xy 190.5 46.99) (xy 190.5 39.37))
-    (stroke (width 0) (type default))
-  )
-  (wire (pts (xy 179.07 30.48) (xy 190.5 30.48))
-    (stroke (width 0) (type default))
-  )
-  (wire (pts (xy 163.83 30.48) (xy 163.83 46.99))
+  (wire (pts (xy 179.07 46.99) (xy 190.5 46.99))
     (stroke (width 0) (type default))
   )
@@
     (stroke (width 0) (type default))
   )
+  (wire (pts (xy 179.07 34.29) (xy 196.85 34.29))
+    (stroke (width 0) (type default))
+  )
   (wire (pts (xy 99.06 80.01) (xy 95.25 80.01))
     (stroke (width 0) (type default))
@@
     (stroke (width 0) (type default))
   )
-  (global_label "latch" (shape input) (at 77.47 64.77 0) (fields_autoplaced)
+  (global_label "keep_alive" (shape input) (at 77.47 64.77 0) (fields_autoplaced)
     (effects (font (size 1.27 1.27)) (justify left))
-    (property "Intersheetrefs" "${INTERSHEET_REFS}" (at 85.2327 64.77 0)
+    (property "Intersheetrefs" "${INTERSHEET_REFS}" (at 90.2523 64.77 0)
       (effects (font (size 1.27 1.27)) (justify left) hide)
     )
   )
-  (global_label "latch" (shape input) (at 176.53 71.12 0) (fields_autoplaced)
+  (global_label "keep_alive" (shape input) (at 176.53 71.12 0) (fields_autoplaced)
     (effects (font (size 1.27 1.27)) (justify left))
-    (property "Intersheetrefs" "${INTERSHEET_REFS}" (at 184.2927 71.12 0)
+    (property "Intersheetrefs" "${INTERSHEET_REFS}" (at 189.3123 71.12 0)
       (effects (font (size 1.27 1.27)) (justify left) hide)
     )
@@
     )
   )
-  (symbol (lib_id "Switch:SW_Push") (at 173.99 30.48 0) (unit 1)
-    (in_bom yes) (on_board yes) (dnp no) (fields_autoplaced)
-    (property "Reference" "SW2" (at 173.99 22.86 0)
-      (effects (font (size 1.27 1.27)))
-    )
-    (property "Value" "next" (at 173.99 25.4 0)
-      (effects (font (size 1.27 1.27)))
-    )
-    (property "Footprint" "" (at 173.99 25.4 0)
-      (effects (font (size 1.27 1.27)) hide)
-    )
-    (property "Datasheet" "~" (at 173.99 25.4 0)
+  (symbol (lib_id "Switch:SW_Push") (at 173.99 46.99 0) (unit 1)
+    (in_bom yes) (on_board yes) (dnp no) (fields_autoplaced)
+    (property "Reference" "SW2" (at 173.99 39.37 0)
+      (effects (font (size 1.27 1.27)))
+    )
+    (property "Value" "next" (at 173.99 41.91 0)
+      (effects (font (size 1.27 1.27)))
+    )
+    (property "Footprint" "" (at 173.99 41.91 0)
+      (effects (font (size 1.27 1.27)) hide)
+    )
+    (property "Datasheet" "~" (at 173.99 41.91 0)
       (effects (font (size 1.27 1.27)) hide)
     )
@@
     )
   )
+  (symbol (lib_id "Switch:SW_Push") (at 173.99 34.29 0) (unit 1)
+    (in_bom yes) (on_board yes) (dnp no) (fields_autoplaced)
+    (property "Reference" "SW3" (at 173.99 26.67 0)
+      (effects (font (size 1.27 1.27)))
+    )
+    (property "Value" "previous" (at 173.99 29.21 0)
+      (effects (font (size 1.27 1.27)))
+    )
+    (property "Footprint" "" (at 173.99 29.21 0)
+      (effects (font (size 1.27 1.27)) hide)
+    )
+    (property "Datasheet" "~" (at 173.99 29.21 0)
+      (effects (font (size 1.27 1.27)) hide)
+    )
+    (pin "1")
+    (pin "2")
+    (instances
+      (project "bam"
+        (path "/81bf8c4d-35fa-42c7-93c2-098e5ef35825"
+          (reference "SW3") (unit 1)
+        )
+      )
+    )
+  )
   (symbol (lib_id "Device:R") (at 105.41 58.42 90) (unit 1)
     (in_bom yes) (on_board yes) (dnp no) (fields_autoplaced)
@@
         (path "/81bf8c4d-35fa-42c7-93c2-098e5ef35825"
           (reference "R2") (unit 1)
-        )
-      )
-    )
-  )
-  (symbol (lib_id "Device:R") (at 182.88 46.99 90) (unit 1)
-    (in_bom yes) (on_board yes) (dnp no) (fields_autoplaced)
-    (property "Reference" "R5" (at 182.88 40.64 90)
-      (effects (font (size 1.27 1.27)))
-    )
-    (property "Value" "33k" (at 182.88 43.18 90)
-      (effects (font (size 1.27 1.27)))
-    )
-    (property "Footprint" "" (at 182.88 48.768 90)
-      (effects (font (size 1.27 1.27)) hide)
-    )
-    (property "Datasheet" "~" (at 182.88 46.99 0)
-      (effects (font (size 1.27 1.27)) hide)
-    )
-    (pin "1")
-    (pin "2")
-    (instances
-      (project "bam"
-        (path "/81bf8c4d-35fa-42c7-93c2-098e5ef35825"
-          (reference "R5") (unit 1)
         )
       )
@@
         )
       )
-    )
-  )
-  (symbol (lib_id "Switch:SW_Push") (at 173.99 46.99 0) (unit 1)
-    (in_bom yes) (on_board yes) (dnp no) (fields_autoplaced)
-    (property "Reference" "SW3" (at 173.99 39.37 0)
-      (effects (font (size 1.27 1.27)))
-    )
-    (property "Value" "play/pause" (at 173.99 41.91 0)
-      (effects (font (size 1.27 1.27)))
-    )
-    (property "Footprint" "" (at 173.99 41.91 0)
-      (effects (font (size 1.27 1.27)) hide)
-    )
-    (property "Datasheet" "~" (at 173.99 41.91 0)
-      (effects (font (size 1.27 1.27)) hide)
-    )
-    (pin "1")
-    (pin "2")
-    (instances
-      (project "bam"
-        (path "/81bf8c4d-35fa-42c7-93c2-098e5ef35825"
-          (reference "SW3") (unit 1)
-        )
-      )
