File: eBoard/eBoard.kicad_sch (KiCad schematic)
At the start: 164 parts, among them Q1 PN2222A, Q2 PN2222A, Q3 PN2222A, Q4 PN2222A, Q5 PN2222A, Q6 PN2222A, Q7 PN2222A, Q8 PN2222A, U1 DRV5055A3xLPGxQ1, U10 DRV5055A3xLPGxQ1, U11 74HC595, U12 74HC595, U13 DRV5055A3xLPGxQ1, U14 DRV5055A3xLPGxQ1, U15 DRV5055A3xLPGxQ1, U16 DRV5055A3xLPGxQ1, U17 DRV5055A3xLPGxQ1, U18 DRV5055A3xLPGxQ1, U19 DRV5055A3xLPGxQ1, U2 74HC595, U20 DRV5055A3xLPGxQ1, U21 DRV5055A3xLPGxQ1, U22 DRV5055A3xLPGxQ1, U23 DRV5055A3xLPGxQ1, U24 DRV5055A3xLPGxQ1, U25 DRV5055A3xLPGxQ1, U26 DRV5055A3xLPGxQ1, U27 DRV5055A3xLPGxQ1, U28 DRV5055A3xLPGxQ1, U29 DRV5055A3xLPGxQ1, U3 DRV5055A3xLPGxQ1, U30 DRV5055A3xLPGxQ1, U31 DRV5055A3xLPGxQ1, U32 DRV5055A3xLPGxQ1, U33 DRV5055A3xLPGxQ1, U34 DRV5055A3xLPGxQ1, U35 DRV5055A3xLPGxQ1, U36 DRV5055A3xLPGxQ1, U37 DRV5055A3xLPGxQ1, U38 DRV5055A3xLPGxQ1, U39 DRV5055A3xLPGxQ1, U4 DRV5055A3xLPGxQ1, U40 DRV5055A3xLPGxQ1, U41 DRV5055A3xLPGxQ1, U42 DRV5055A3xLPGxQ1, U43 DRV5055A3xLPGxQ1, U44 DRV5055A3xLPGxQ1, U45 DRV5055A3xLPGxQ1, U46 DRV5055A3xLPGxQ1, U47 DRV5055A3xLPGxQ1, U48 DRV5055A3xLPGxQ1, U49 DRV5055A3xLPGxQ1, U5 DRV5055A3xLPGxQ1, U50 DRV5055A3xLPGxQ1, U51 DRV5055A3xLPGxQ1, U52 DRV5055A3xLPGxQ1, U53 DRV5055A3xLPGxQ1, U54 DRV5055A3xLPGxQ1, U55 DRV5055A3xLPGxQ1, U56 DRV5055A3xLPGxQ1, U57 DRV5055A3xLPGxQ1, U58 DRV5055A3xLPGxQ1, U59 DRV5055A3xLPGxQ1, U6 DRV5055A3xLPGxQ1, U60 DRV5055A3xLPGxQ1, U61 DRV5055A3xLPGxQ1, U62 DRV5055A3xLPGxQ1, U63 DRV5055A3xLPGxQ1, U64 DRV5055A3xLPGxQ1, U65 DRV5055A3xLPGxQ1, U66 DRV5055A3xLPGxQ1, U67 DRV5055A3xLPGxQ1, U7 DRV5055A3xLPGxQ1, U8 DRV5055A3xLPGxQ1, U9 DRV5055A3xLPGxQ1

Commit message: eboard wip
Parts:
- added D65, D66, D67, D68: 1N5711, Diode_THT:D_DO-35_SOD27_P7.62mm_Horizontal, symbol Diode:1N5711
- added Q10, Q11, Q12, Q9: PN2222A, Package_TO_SOT_THT:TO-92_Inline, symbol Transistor_BJT:PN2222A
- added R17: 1k, symbol Device:R
- added R18, R20: R, symbol Device:R
- added R19, R21: 10k, symbol Device:R
- added U68, U69, U70, U71: DRV5055A3xLPGxQ1, Package_TO_SOT_SMD:SOT-23W_Handsoldering, symbol Sensor_Magnetic:DRV5055A3xLPGxQ1
Connections:
- net GND: now also U68.2 (GND), U69.2 (GND), U70.2 (GND), U71.2 (GND)
- net Vcc: now also U68.1 (VCC), U69.1 (VCC), U70.1 (VCC), U71.1 (VCC)
- new net: Q11.1 (E), Q9.1 (E), R17.1
- new net: Q9.2 (B), R19.1
- new net: D66.1 (K), Q9.3 (C)
- new net: D68.2 (A), U71.3 (OUT)
- new net: R19.2, R21.2
- new net: Q11.2 (B), Q12.2 (B), R20.2
- new net: D67.1 (K), Q11.3 (C)
- new net: D65.1 (K), Q10.3 (C)
- new net: D65.2 (A), U69.3 (OUT)
- new net: D67.2 (A), U70.3 (OUT)
- new net: D68.1 (K), Q12.3 (C)
- new net: D66.2 (A), U68.3 (OUT)
- new net: Q10.1 (E), Q12.1 (E), R18.1
- new net: Q10.2 (B), R21.1

Commit message: update
Parts:
- removed D65, D66, D67, D68: 1N5711, Diode_THT:D_DO-35_SOD27_P7.62mm_Horizontal, symbol Diode:1N5711
- removed R20: R, symbol Device:R
- added R22, R23: 10k, symbol Device:R
- R17: value 1k -> 10k
- R18: value R -> 10k
Connections:
- net A0: now also Q11.1 (E), Q9.1 (E), R17.1
- net A1: now also Q10.1 (E), Q12.1 (E), R18.1
- net GND: now also R17.2, R18.2
- net at Q9.3 (C): now also U68.3 (OUT)
- net at U71.3 (OUT): now also Q12.3 (C)
- net at Q11.2 (B): now also R22.1; no longer Q12.2 (B)
- net at Q11.3 (C): now also U70.3 (OUT)
- net at Q10.3 (C): now also U69.3 (OUT)
- new net: Q12.2 (B), R23.1
- new net: R22.2, R23.2

Commit message: wip
Parts:
- removed C1, C2, C3, C4, C5, C6, C7, C8: C, symbol Device:C
- removed Q1, Q2, Q3, Q4, Q5, Q6, Q7, Q8: PN2222A, Package_TO_SOT_THT:TO-92_Inline, symbol Transistor_BJT:PN2222A
- removed R10, R11, R12, R13, R14, R15, R16, R9: 10k, symbol Device:R
- removed U1, U10, U13, U14, U15, U16, U17, U18, U19, U20, U21, U22, U23, U24, U25, U26, U27, U28, U29, U3, U30, U31, U32, U33, U34, U35, U36, U37, U38, U39, U4, U40, U41, U42, U43, U44, U45, U46, U47, U48, U49, U5, U50, U51, U52, U53, U54, U55, U56, U57, U58, U59, U6, U60, U61, U62, U63, U64, U65, U66, U67, U7, U8, U9: DRV5055A3xLPGxQ1, Package_TO_SOT_SMD:SOT-23W_Handsoldering, symbol Sensor_Magnetic:DRV5055A3xLPGxQ1
Connections:
- net at U2.15 (QA): now also R19.2, R21.2
- net at U2.1 (QB): now also R22.2, R23.2
Other:
- moved on the sheet: Q10, Q11, Q12, Q9, R17, R18, R19, R21, R22, R23, U68, U69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
